File: hardware/CAN SPE CARRIER/CAN SPE CARRIER.kicad_pcb (KiCad board)
At the start: 2 copper layers, 18 parts, among them J1 Screw_Terminal_01x03, J2 Conn_01x02, J3 Conn_01x08, J4 Conn_01x08, J5 Conn_02x35_Odd_Even, J6 Conn_02x35_Odd_Even, U2 MCP2562FDT-H_SN

Commit message: [Updated]: Updated the PCB Design
Parts:
- J5, J6: moved to B.Cu
- moved U2 71.8 mm to (36.4, 120.1)
- moved C2 70.6 mm to (29.9, 120.5), turned to 90 degrees
- moved J5 67.9 mm to (21.9, 50.0), turned to 180 degrees
- moved TP1 67.1 mm to (46.8, 76.3)
- moved R3 64.0 mm to (52.5, 77.0), turned to 90 degrees
- moved J1 63.5 mm to (72.2, 120.8), turned to 180 degrees
- moved D1 61.1 mm to (52.5, 73.3), turned to -90 degrees
- moved C1 60.6 mm to (42.0, 125.2), turned to -90 degrees
- moved TP2 58.0 mm to (52.0, 88.0)
- moved R2 53.0 mm to (64.1, 77.1), turned to -90 degrees
- moved J4 48.0 mm to (59.0, 50.0), turned to 90 degrees
- moved C4 47.7 mm to (70.5, 77.3), turned to 90 degrees
- moved C3 47.6 mm to (60.0, 85.6), turned to -90 degrees
- moved D2 45.8 mm to (68.2, 128.5), turned to 90 degrees
- moved R1 43.0 mm to (68.2, 133.0)
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Routing:
- net +5V: track 0.00 -> 164.6 mm, vias 0 -> 1
- net +3V3: track 0.00 -> 122.9 mm, vias 0 -> 2
- net /SPI_MOSI: track 0.00 -> 61.1 mm
- net /SPI_SCK: track 0.00 -> 57.0 mm
- net /SPI_MISO: track 0.00 -> 57.0 mm
- net Net-(J1-Pin_1): track 0.00 -> 54.6 mm
- net /SPI_CS: track 0.00 -> 54.2 mm
- net /MB_RST: track 0.00 -> 49.0 mm
- net Net-(J1-Pin_2): track 0.00 -> 47.9 mm
- net /MB_INT: track 0.00 -> 32.1 mm
- net /MB_SCL: track 0.00 -> 22.5 mm
- net /MB_SDA: track 0.00 -> 20.9 mm
- net /CAN_TX: track 0.00 -> 12.9 mm
- net /CAN_RX: track 0.00 -> 12.7 mm
- net GND: track 0.00 -> 6.05 mm, vias 0 -> 2
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- added copper zone on B.Cu, net GND
- added copper zone on F.Cu, net GND
Other:
- board outline added: 70 x 94.2 mm
